File: AB_shield.brd (EAGLE design)
At the start: 68.6 x 53.3 mm, 11 parts, among them U1 ARDUINOR3-DIMENSION, X2 MOTOR

Commit message: update
Routing:
- net N$9: track 38.5 -> 32.4 mm
- net N$10: track 48.7 -> 44.1 mm
Changed lines of the file:
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@@
 <contactref element="AB_OUT" pad="2"/>
 <contactref element="X2" pad="3"/>
-<wire x1="26.67" y1="20.32" x2="25.4" y2="19.05" width="1.27" layer="16"/>
-<wire x1="25.4" y1="19.05" x2="22.86" y2="19.05" width="1.27" layer="16"/>
-<wire x1="26.67" y1="20.32" x2="26.67" y2="29.21" width="1.27" layer="16"/>
-<wire x1="26.67" y1="29.21" x2="24.765" y2="31.115" width="1.27" layer="16"/>
-<wire x1="24.765" y1="31.115" x2="13.97" y2="31.115" width="1.27" layer="16"/>
-<wire x1="13.97" y1="31.115" x2="6.985" y2="38.1" width="1.27" layer="16"/>
 <wire x1="6.985" y1="38.1" x2="5.1054" y2="38.1" width="1.27" layer="16"/>
 <wire x1="5.1054" y1="38.1" x2="5.08" y2="38.0492" width="1.27" layer="16"/>
+<wire x1="22.86" y1="19.05" x2="18.415" y2="19.05" width="1.27" layer="1"/>
+<wire x1="18.415" y1="19.05" x2="9.525" y2="27.94" width="1.27" layer="1"/>
+<wire x1="9.525" y1="27.94" x2="9.525" y2="36.195" width="1.27" layer="1"/>
+<wire x1="9.525" y1="36.195" x2="7.6708" y2="38.0492" width="1.27" layer="1"/>
+<wire x1="7.6708" y1="38.0492" x2="5.08" y2="38.0492" width="1.27" layer="1"/>
 </signal>
 <signal name="N$10">
 <contactref element="AB_OUT" pad="1"/>
 <contactref element="X2" pad="4"/>
-<wire x1="22.86" y1="16.51" x2="27.94" y2="16.51" width="1.27" layer="16"/>
-<wire x1="27.94" y1="16.51" x2="29.21" y2="17.78" width="1.27" layer="16"/>
-<wire x1="29.21" y1="17.78" x2="29.21" y2="29.845" width="1.27" layer="16"/>
 <wire x1="5.207" y1="43.18" x2="5.08" y2="43.0784" width="1.27" layer="16"/>
-<wire x1="29.21" y1="29.845" x2="26.035" y2="33.02" width="1.27" layer="16"/>
-<wire x1="26.035" y1="33.02" x2="15.113" y2="33.02" width="1.27" layer="16"/>
-<wire x1="15.113" y1="33.02" x2="5.08" y2="43.0784" width="1.27" layer="16"/>
+<wire x1="5.08" y1="43.0784" x2="4.3434" y2="43.0784" width="1.27" layer="1"/>
+<wire x1="4.3434" y1="43.0784" x2="1.905" y2="40.64" width="1.27" layer="1"/>
+<wire x1="1.905" y1="40.64" x2="1.905" y2="26.67" width="1.27" layer="1"/>
+<wire x1="1.905" y1="26.67" x2="6.985" y2="21.59" width="1.27" layer="1"/>
+<wire x1="6.985" y1="21.59" x2="10.795" y2="21.59" width="1.27" layer="1"/>
+<wire x1="10.795" y1="21.59" x2="15.875" y2="16.51" width="1.27" layer="1"/>
+<wire x1="15.875" y1="16.51" x2="22.86" y2="16.51" width="1.27" layer="1"/>
+<wire x1="23.495" y1="16.51" x2="22.86" y2="16.51" width="1.27" layer="1"/>
 </signal>
 <signal name="N$11">

Commit message: Added silkscreen pinout and jumper info
Parts:
- JP1: value USE_VIN -> (none)
- X2: value MOTOR -> (none)
Other:
- outline, holes or cut-outs redrawn
- board text added: "Default"
- board text added: "GND"
- board text added: "MOT1A"
- board text added: "MOT1B"
- board text added: "MOT2A"
- board text added: "MOT2B"
- board text added: "Use Vin pin as VMOT"
- board text added: "VMOT"
Changed lines of the file:
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@@
 <rectangle x1="19.05" y1="34.29" x2="62.23" y2="46.99" layer="41"/>
 <rectangle x1="19.05" y1="34.29" x2="62.23" y2="46.99" layer="42"/>
+<text x="9.525" y="32.385" size="1.778" layer="21">MOT2A</text>
+<text x="9.525" y="27.305" size="1.778" layer="21">MOT2B</text>
+<text x="9.525" y="36.83" size="1.778" layer="21">MOT1A</text>
+<text x="9.525" y="41.91" size="1.778" layer="21">MOT1B</text>
+<text x="13.97" y="12.7" size="1.778" layer="21">GND</text>
+<text x="13.335" y="17.145" size="1.778" layer="21">VMOT</text>
+<wire x1="27.305" y1="9.525" x2="29.21" y2="9.525" width="0.4064" layer="21"/>
+<wire x1="31.115" y1="9.525" x2="33.02" y2="9.525" width="0.4064" layer="21"/>
+<wire x1="33.02" y1="9.525" x2="33.02" y2="12.065" width="0.4064" layer="21"/>
+<wire x1="33.02" y1="12.065" x2="31.115" y2="12.065" width="0.4064" layer="21"/>
+<wire x1="31.115" y1="12.065" x2="29.21" y2="12.065" width="0.4064" layer="21"/>
+<wire x1="29.21" y1="12.065" x2="27.305" y2="12.065" width="0.4064" layer="21"/>
+<wire x1="27.305" y1="12.065" x2="27.305" y2="9.525" width="0.4064" layer="21"/>
+<wire x1="29.21" y1="12.065" x2="29.21" y2="9.525" width="0.4064" layer="21"/>
+<wire x1="29.21" y1="9.525" x2="31.115" y2="9.525" width="0.4064" layer="21"/>
+<wire x1="31.115" y1="9.525" x2="31.115" y2="12.065" width="0.4064" layer="21"/>
+<rectangle x1="27.94" y1="10.16" x2="30.48" y2="11.43" layer="21"/>
+<wire x1="27.305" y1="5.715" x2="29.21" y2="5.715" width="0.4064" layer="21"/>
+<wire x1="31.115" y1="5.715" x2="33.02" y2="5.715" width="0.4064" layer="21"/>
+<wire x1="33.02" y1="5.715" x2="33.02" y2="8.255" width="0.4064" layer="21"/>
+<wire x1="33.02" y1="8.255" x2="31.115" y2="8.255" width="0.4064" layer="21"/>
+<wire x1="31.115" y1="8.255" x2="29.21" y2="8.255" width="0.4064" layer="21"/>
+<wire x1="29.21" y1="8.255" x2="27.305" y2="8.255" width="0.4064" layer="21"/>
+<wire x1="27.305" y1="8.255" x2="27.305" y2="5.715" width="0.4064" layer="21"/>
+<wire x1="29.21" y1="8.255" x2="29.21" y2="5.715" width="0.4064" layer="21"/>
+<wire x1="29.21" y1="5.715" x2="31.115" y2="5.715" width="0.4064" layer="21"/>
+<wire x1="31.115" y1="5.715" x2="31.115" y2="8.255" width="0.4064" layer="21"/>
+<rectangle x1="29.845" y1="6.35" x2="32.385" y2="7.62" layer="21"/>
+<text x="34.29" y="6.35" size="1.27" layer="21">Use Vin pin as VMOT</text>
+<text x="34.29" y="10.16" size="1.27" layer="21">Default</text>
+<circle x="13.97" y="2.54" radius="1.79605" width="0.3048" layer="20"/>
+<circle x="66.04" y="7.62" radius="1.79605" width="0.3048" layer="20"/>
+<circle x="66.04" y="35.56" radius="1.79605" width="0.3048" layer="20"/>
+<circle x="15.24" y="50.8" radius="1.79605" width="0.3048" layer="20"/>
 </plain>
 <attributes>
@@
 <attribute name="OC_FARNELL" value="unknown" x="60.96" y="22.86" size="1.778" layer="27" rot="R270" display="off"/>
 </element>
-<element name="AB_OUT" library="con-lstb" package="MA06-1" value="" x="22.86" y="22.86" rot="R90">
+<element name="AB_OUT" library="con-lstb" package="MA06-1" value="" x="22.86" y="22.86" smashed="yes" rot="R90">
 <attribute name="MF" value="" x="22.86" y="22.86" size="1.778" layer="27" rot="R90" display="off"/>
 <attribute name="OC_NEWARK" value="unknown" x="22.86" y="22.86" size="1.778" layer="27" rot="R90" display="off"/>
 <attribute name="MPN" value="" x="22.86" y="22.86" size="1.778" layer="27" rot="R90" display="off"/>
 <attribute name="OC_FARNELL" value="unknown" x="22.86" y="22.86" size="1.778" layer="27" rot="R90" display="off"/>
-</element>
-<element name="JP1" library="jumper" package="JP2" value="USE_VIN" x="22.86" y="7.62" rot="R180"/>
+<attribute name="NAME" x="26.924" y="22.86" size="1.27" layer="25" ratio="10" rot="R90"/>
+<attribute name="VALUE" x="25.781" y="20.32" size="1.27" layer="27" ratio="10" rot="R90"/>
+</element>
+<element name="JP1" library="jumper" package="JP2" value="" x="22.86" y="7.62" rot="R180"/>
 <element name="X1" library="con-ptr500" package="AK500/2-H" value="" x="5.08" y="15.24" smashed="yes" rot="R90">
 <attribute name="MF" value="" x="5.08" y="15.24" size="1.778" layer="27" rot="R90" display="off"/>
@@
 <attribute name="VALUE" x="14.605" y="10.16" size="1.778" layer="27" ratio="10" rot="R90"/>
 </element>
-<element name="X2" library="con-ptr500" package="AK500/4" value="MOTOR" x="5.08" y="35.56" smashed="yes" rot="R90">
+<element name="X2" library="con-ptr500" package="AK500/4" value="" x="5.08" y="35.56" smashed="yes" rot="R90">
 <attribute name="MF" value="" x="5.08" y="35.56" size="1.778" layer="27" rot="R90" display="off"/>
 <attribute name="OC_NEWARK" value="unknown" x="5.08" y="35.56" size="1.778" layer="27" rot="R90" display="off"/>
@@
 <attribute name="OC_FARNELL" value="unknown" x="5.08" y="35.56" size="1.778" layer="27" rot="R90" display="off"/>
 <attribute name="NAME" x="4.3688" y="47.625" size="1.778" layer="25" ratio="10" rot="R180"/>
-<attribute name="VALUE" x="10.795" y="25.4762" size="1.778" layer="27" ratio="10" rot="R90"/>
+<attribute name="VALUE" x="7.62" y="45.7962" size="1.778" layer="27" ratio="10" rot="R90"/>
 </element>
 <element name="U1" library="adafruit" package="ARDUINOR3" value="ARDUINOR3-DIMENSION" x="0" y="0"/>
